File: MCU_Datalogger.kicad_sch (KiCad schematic)
At the start: 25 parts, among them U1 24LC1025, U2 24LC1025, U3 DS1337S_, U4 ATMEGA328P-AN, Y1 16 MHz, Y2 32.768 KHz

Commit message: Completed Comments
Other:
- note added: "MCU"
- note added: "Memory EEPROM"
- note added: "Mounting"
- note added: "Real Time CLock"
Changed lines of the file:
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@@
 	(wire
 		(pts
-			(xy 166.37 118.11) (xy 153.67 118.11)
+			(xy 177.8 118.11) (xy 165.1 118.11)
 		)
 		(stroke
@@
 	(wire
 		(pts
-			(xy 153.67 114.3) (xy 166.37 114.3)
+			(xy 165.1 114.3) (xy 177.8 114.3)
 		)
 		(stroke
@@
 	(wire
 		(pts
-			(xy 153.67 118.11) (xy 153.67 120.65)
+			(xy 165.1 118.11) (xy 165.1 120.65)
 		)
 		(stroke
@@
 		)
 	)
+	(rectangle
+		(start 235.585 113.665)
+		(end 266.065 154.94)
+		(stroke
+			(width 0)
+			(type default)
+		)
+		(fill
+			(type none)
+		)
+	)
+	(rectangle
+		(start 26.67 114.935)
+		(end 139.7 161.925)
+		(stroke
+			(width 0)
+			(type default)
+		)
+		(fill
+			(type none)
+		)
+	)
+	(rectangle
+		(start 135.255 19.05)
+		(end 281.94 97.155)
+		(stroke
+			(width 0)
+			(type default)
+		)
+		(fill
+			(type none)
+		)
+	)
+	(rectangle
+		(start 20.955 23.495)
+		(end 128.27 92.71)
+		(stroke
+			(width 0)
+			(type default)
+		)
+		(fill
+			(type none)
+		)
+	)
+	(text "Real Time CLock"
+		(exclude_from_sim no)
+		(at 28.956 22.098 0)
+		(effects
+			(font
+				(size 1.27 1.27)
+			)
+		)
+	)
+	(text "Mounting"
+		(exclude_from_sim no)
+		(at 239.522 112.268 0)
+		(effects
+			(font
+				(size 1.27 1.27)
+			)
+		)
+	)
+	(text "Memory EEPROM"
+		(exclude_from_sim no)
+		(at 35.052 113.538 0)
+		(effects
+			(font
+				(size 1.27 1.27)
+			)
+		)
+	)
+	(text "MCU\n"
+		(exclude_from_sim no)
+		(at 137.414 17.78 0)
+		(effects
+			(font
+				(size 1.27 1.27)
+			)
+		)
+	)
 	(label "SCK"
 		(at 97.79 140.97 0)
@@
 	)
 	(label "D2"
-		(at 194.31 116.84 0)
+		(at 205.74 116.84 0)
 		(fields_autoplaced yes)
 		(effects
@@
 	)
 	(label "Vcc"
-		(at 153.67 114.3 180)
+		(at 165.1 114.3 180)
 		(fields_autoplaced yes)
 		(effects
@@
 	)
 	(label "D7"
-		(at 194.31 135.89 0)
+		(at 205.74 135.89 0)
 		(fields_autoplaced yes)
 		(effects
@@
 	)
 	(label "SCK"
-		(at 166.37 129.54 180)
+		(at 177.8 129.54 180)
 		(fields_autoplaced yes)
 		(effects
@@
 	)
 	(label "D3"
-		(at 194.31 120.65 0)
+		(at 205.74 120.65 0)
 		(fields_autoplaced yes)
 		(effects
@@
 	)
 	(label "SDA"
-		(at 166.37 125.73 180)
+		(at 177.8 125.73 180)
 		(fields_autoplaced yes)
 		(effects
@@
 	)
 	(label "D4"
-		(at 194.31 124.46 0)
+		(at 205.74 124.46 0)
 		(fields_autoplaced yes)
 		(effects
@@
 	)
 	(label "MISO"
-		(at 166.37 151.13 180)
+		(at 177.8 151.13 180)
 		(fields_autoplaced yes)
 		(effects
@@
 	)
 	(label "D6"
-		(at 194.31 132.08 0)
+		(at 205.74 132.08 0)
 		(fields_autoplaced yes)
 		(effects
@@
 	)
 	(label "MOSI"
-		(at 166.37 147.32 180)
+		(at 177.8 147.32 180)
 		(fields_autoplaced yes)
 		(effects
@@
 	)
 	(label "D8"
-		(at 194.31 139.7 0)
+		(at 205.74 139.7 0)
 		(fields_autoplaced yes)
 		(effects
@@
 	)
 	(label "RESET"
-		(at 194.31 151.13 0)
+		(at 205.74 151.13 0)
 		(fields_autoplaced yes)
 		(effects
@@
 	)
 	(label "D5"
-		(at 194.31 128.27 0)
+		(at 205.74 128.27 0)
 		(fields_autoplaced yes)
 		(effects
@@
 	)
 	(label "RX"
-		(at 166.37 137.16 180)
+		(at 177.8 137.16 180)
 		(fields_autoplaced yes)
 		(effects
@@
 	)
 	(label "TX"
-		(at 166.37 140.97 180)
+		(at 177.8 140.97 180)
 		(fields_autoplaced yes)
 		(effects
@@
 	(symbol
 		(lib_id "power:GND")
-		(at 153.67 120.65 0)
+		(at 165.1 120.65 0)
 		(unit 1)
 		(exclude_from_sim no)
@@
 		(fields_autoplaced yes)
 		(property "Reference" "#PWR010"
-			(at 153.67 127 0)
+			(at 165.1 127 0)
 			(effects
 				(font
@@
 		)
 		(property "Value" "GND"
-			(at 153.67 125.73 0)
+			(at 165.1 125.73 0)
 			(effects
 				(font
@@
 		)
 		(property "Footprint" ""
-			(at 153.67 120.65 0)
+			(at 165.1 120.65 0)
 			(effects
 				(font
@@
 		)
 		(property "Datasheet" ""
-			(at 153.67 120.65 0)
+			(at 165.1 120.65 0)
 			(effects
 				(font
@@
 		)
 		(property "Description" "Power symbol creates a global label with name \"GND\" , ground"
-			(at 153.67 120.65 0)
+			(at 165.1 120.65 0)
 			(effects
 				(font
@@
 	)
 	(sheet
-		(at 166.37 109.22)
+		(at 177.8 109.22)
 		(size 27.94 46.99)
 		(fields_autoplaced yes)
@@
 		)
 		(property "Sheetname" "Connectors"
-			(at 166.37 108.5084 0)
+			(at 177.8 108.5084 0)
 			(effects
 				(font
@@
 		)
 		(property "Sheetfile" "connectors.kicad_sch"
-			(at 166.37 156.7946 0)
+			(at 177.8 156.7946 0)
 			(effects
 				(font
@@
 		)
 		(pin "D4" bidirectional
-			(at 194.31 124.46 0)
+			(at 205.74 124.46 0)
 			(effects
 				(font
@@
 		)
 		(pin "D2" bidirectional
-			(at 194.31 116.84 0)
+			(at 205.74 116.84 0)
 			(effects
 				(font
@@
 		)
 		(pin "D3" bidirectional
-			(at 194.31 120.65 0)
+			(at 205.74 120.65 0)
 			(effects
 				(font
@@
 		)
 		(pin "D5" bidirectional
-			(at 194.31 128.27 0)
+			(at 205.74 128.27 0)
 			(effects
 				(font
@@
 		)
 		(pin "GND" passive
-			(at 166.37 118.11 180)
+			(at 177.8 118.11 180)
 			(effects
 				(font
@@
 		)
 		(pin "RX" input
-			(at 166.37 137.16 180)
+			(at 177.8 137.16 180)
 			(effects
 				(font
@@
 		)
 		(pin "TX" output
-			(at 166.37 140.97 180)
+			(at 177.8 140.97 180)
 			(effects
 				(font
@@
 		)
 		(pin "Vcc" passive
-			(at 166.37 114.3 180)
+			(at 177.8 114.3 180)
 			(effects
 				(font
@@
 		)
 		(pin "SCK" passive
-			(at 166.37 129.54 180)
+			(at 177.8 129.54 180)
 			(effects
 				(font
@@
 		)
 		(pin "SDA" bidirectional
-			(at 166.37 125.73 180)
+			(at 177.8 125.73 180)
 			(effects
 				(font
@@
 		)
 		(pin "D7" bidirectional
-			(at 194.31 135.89 0)
+			(at 205.74 135.89 0)
 			(effects
 				(font
@@
 		)
 		(pin "D6" bidirectional
-			(at 194.31 132.08 0)
+			(at 205.74 132.08 0)
 			(effects
 				(font
@@
 		)
 		(pin "D8" bidirectional
-			(at 194.31 139.7 0)
+			(at 205.74 139.7 0)
 			(effects
 				(font
@@
 		)
 		(pin "MOSI" input
-			(at 166.37 147.32 180)
+			(at 177.8 147.32 180)
 			(effects
 				(font
@@
 		)
 		(pin "MISO" output
-			(at 166.37 151.13 180)
+			(at 177.8 151.13 180)
 			(effects
 				(font
@@
 		)
 		(pin "RESET" passive
-			(at 194.31 151.13 0)
+			(at 205.74 151.13 0)
 			(effects
 				(font
